Commit message: initial commit

File: robots/kobuki_hexagons_kinect_multi_robot.urdf.xacro (robot description, xacro)
@@ -11,6 +11,12 @@
   <xacro:include filename="$(find turtlebot_description)/urdf/stacks/hexagons.urdf.xacro"/>
   <xacro:include filename="$(find turtlebot_description)/urdf/sensors/kinect.urdf.xacro"/>
+  <!-- Added -->
+  <xacro:include filename="$(find icclab_turtlebot)/sensors/rplidar.urdf.xacro" />
   <kobuki/>
   <stack_hexagons parent="base_link"/>
   <sensor_kinect  parent="base_link"/>
+<!-- Added -->
+  <xacro:rplidar name="rplidar" parent="base_link" ros_topic="scan" update_rate="5" ray_count="1040" min_angle="0" max_angle="360">
+    <origin xyz="0.1 0 0.420" rpy="3.1415 0 3.1415"/>
+  </xacro:rplidar>
 </robot>
